File: kicad/board-routed_rounded.kicad_pcb (KiCad board)
At the start: 2 copper layers, 140.2 x 108.1 mm, 41 parts

Commit message: Owl
Parts:
- added REF**: MountingHole_3.2mm_M3, mounting holes:MountingHole_3.2mm_M3, F.Cu at (167.2, -107.0)
- added REF**: MountingHole_3.2mm_M3, mounting holes:MountingHole_3.2mm_M3, F.Cu at (47.6, -93.6)
- added REF**: MountingHole_3.2mm_M3, mounting holes:MountingHole_3.2mm_M3, F.Cu at (167.2, -48.2)
- added REF**: MountingHole_3.2mm_M3, mounting holes:MountingHole_3.2mm_M3, F.Cu at (47.6, -53.6)
- moved T1 5.23 mm to (167.6, -73.3)
- moved T2 5.23 mm to (167.6, -73.3)
- moved B1 5.09 mm to (167.0, -59.3)
Routing:
- net Braw: track 51.9 -> 62.4 mm
- net Bplus: track 58.9 -> 69.4 mm
- net RST: track 72.3 -> 77.1 mm
Other:
- board size 140.2 x 108.1 mm -> 140.2 x 108.7 mm
- board text added: "Owl by sapristi remix of rae-dux v0.1 by ajrae"
- board text removed: "rae-dux v0.1 by ajrae"
